File: Hardware/KIM Board/Rev 1.0/KIM Board.kicad_sch (KiCad schematic)
At the start: 87 parts, among them J15 PORT B, J16 PORT A, J23 CART, J24 BUS, J26 DB9 MALE (DTE), J27 CTS EN, J28 DCD EN, J29 5V DC, J30 VCC, J31 POWER LED, SW68 POWER, SW69 IO ENABLE, U10 AT28C256, U11 74HC00, U13 65C22, U14 74HC00, U16 74HC00, U17 74HC00, U18 74HC30, U19 74HC138, U23 74HC00, U28 65C51, U29 MAX238xNG+, U8 65C02, U9 AS6C62256, X2 1MHz, Y1 1.8432 Mhz

Commit message: Finish Keypad Expander layout
Parts:
- removed C21, C23, C25, C27, C29, C31, C33, C35, C37, C39, C41: 100nF, Capacitor_THT:C_Disc_D5.0mm_W2.5mm_P2.50mm, symbol Device:C
- removed J15: PORT B, 6502 Parts:6502 GPIO Connector, symbol Connector_Generic:Conn_02x06_Odd_Even
- removed J16: PORT A, 6502 Parts:6502 GPIO Connector, symbol Connector_Generic:Conn_02x06_Odd_Even
- removed R21, R22, R23, R24, R26, R27, R28, R37, R38, R39, R40, R41, R42, R43, R44, R45: 1k, Resistor_THT:R_Axial_DIN0204_L3.6mm_D1.6mm_P5.08mm_Horizontal, symbol Device:R
- removed U13: 65C22, Package_DIP:DIP-40_W15.24mm_Socket_LongPads, symbol 6502 Parts:65C22
- removed U17, U23: 74HC00, Package_DIP:DIP-14_W7.62mm_Socket_LongPads, symbol 74xx:74HC00
- removed U18: 74HC30, Package_DIP:DIP-14_W7.62mm_Socket_LongPads, symbol 6502 Parts:74HC30
- added C12: 100nF, Capacitor_THT:C_Disc_D5.0mm_W2.5mm_P2.50mm, symbol Device:C
- added J4: PORT B, 6502 Parts:6502 GPIO Connector, symbol Connector_Generic:Conn_02x06_Odd_Even
- added J5: PORT A, 6502 Parts:6502 GPIO Connector, symbol Connector_Generic:Conn_02x06_Odd_Even
- added R16, R17: 1k, Resistor_THT:R_Axial_DIN0204_L3.6mm_D1.6mm_P5.08mm_Horizontal, symbol Device:R
- added SW3: KEYPAD ENBL, 6502 Parts:EG2201A, symbol Switch:SW_Push_DPDT
- added U10: 65C21, Package_DIP:DIP-40_W15.24mm_Socket_LongPads, symbol 6502 Parts:65C21
- added U8: AT28C64, Package_DIP:DIP-28_W15.24mm_Socket_LongPads, symbol 6502 Parts:AT28C64
- added U9: 74HC138, Package_DIP:DIP-16_W7.62mm_Socket_LongPads, symbol 74xx:74HC138
- renumbered C20 to C1, C38 to C10, C40 to C11, C16 to C13, C17 to C14, C18 to C15, C19 to C16, C22 to C2, C24 to C3, C26 to C4, C28 to C5, C30 to C6, C32 to C7, C34 to C8, C36 to C9, D5 to D1, J29 to J1, J28 to J10, J30 to J2, J31 to J3, J23 to J6, J24 to J7, J26 to J8, J27 to J9, R25 to R1, R33 to R10, R19 to R11, R34 to R12, R35 to R13, R36 to R14, R50 to R15, R29 to R2, R15 to R3, R30 to R4, R16 to R5, R31 to R6, R17 to R7, R32 to R8, R18 to R9, SW69 to SW1, SW68 to SW2, TP4 to TP1, TP5 to TP2, U16 to U1, U28 to U11, U29 to U12, U8 to U2, U9 to U3, U14 to U4, U19 to U5, U11 to U6, U10 to U7, X2 to X1
Connections:
- net A0: now also U10.36 (RS0), U8.10 (A0)
- net A1: now also U10.35 (RS1), U8.9 (A1)
- net A10: now also U8.21 (A10)
- net A11: now also U8.23 (A11)
- net A12: now also U8.2 (A12)
- net A13: now also U9.1 (A0)
- net A14: now also U9.2 (A1)
- net A15: now also U9.3 (A2)
- net A2: now also U8.8 (A2)
- net A3: now also U8.7 (A3)
- net A4: now also U8.6 (A4)
- net A5: now also U8.5 (A5)
- net A6: now also U8.4 (A6)
- net A7: now also U8.3 (A7)
- net A8: now also U8.25 (A8)
- net A9: now also U8.24 (A9)
- net CA1: now also J5.11 (Pin_11), U10.40 (CA1)
- net CA2: now also J5.12 (Pin_12), U10.39 (CA2)
- net CB1: now also J4.11 (Pin_11), U10.18 (CB1)
- net CB2: now also J4.12 (Pin_12), U10.19 (CB2)
- net D0: now also U10.33 (D0), U8.11 (I/O0)
- net D1: now also U10.32 (D1), U8.12 (I/O1)
- net D2: now also U10.31 (D2), U8.13 (I/O2)
- net D3: now also U10.30 (D3), U8.15 (I/O3)
- net D4: now also U10.29 (D4), U8.16 (I/O4)
- net D5: now also U10.28 (D5), U8.17 (I/O5)
- net D6: now also U10.27 (D6), U8.18 (I/O6)
- net D7: now also U10.26 (D7), U8.19 (I/O7)
- net GND: now also C12.2, J4.2 (Pin_2), J5.2 (Pin_2), U10.1 (VSS), U8.14 (GND), U9.4 (~{E0}), U9.5 (~{E1}), U9.8 (GND)
- net IRQB: now also U10.37 (IRQBB), U10.38 (IRQAB)
- net PA0: now also J5.4 (Pin_4), U10.2 (PA0)
- net PA1: now also J5.6 (Pin_6), U10.3 (PA1)
- net PA2: now also J5.8 (Pin_8), U10.4 (PA2)
- net PA3: now also J5.10 (Pin_10), U10.5 (PA3)
- net PA4: now also J5.9 (Pin_9), U10.6 (PA4)
- net PA5: now also J5.7 (Pin_7), U10.7 (PA5)
- net PA6: now also J5.5 (Pin_5), U10.8 (PA6)
- net PA7: now also J5.3 (Pin_3), U10.9 (PA7)
- net PB0: now also J4.4 (Pin_4), U10.10 (PB0)
- net PB1: now also J4.6 (Pin_6), U10.11 (PB1)
- net PB2: now also J4.8 (Pin_8), U10.12 (PB2)
- net PB3: now also J4.10 (Pin_10), U10.13 (PB3)
- net PB4: now also J4.9 (Pin_9), U10.14 (PB4)
- net PB5: now also J4.7 (Pin_7), U10.15 (PB5)
- net PB6: now also J4.5 (Pin_5), U10.16 (PB6)
- net PB7: now also J4.3 (Pin_3), U10.17 (PB7)
- net PHI2: now also U10.25 (PHI2)
- net RB: now also U8.22 (~{OE})
- net REB: now also R17.1, SW3.4 (A), U8.20 (~{CE})
- net RESB: now also U10.34 (RESB)
- net RWB: now also U10.21 (RWB)
- net VCC: now also C12.1, J4.1 (Pin_1), J5.1 (Pin_1), R16.2, R17.2, U10.20 (VDD), U10.22 (CS0), U10.24 (CS1), U8.27 (~{WE}), U8.28 (VCC), U9.16 (VCC), U9.6 (E2)
- new net: SW3.5 (B), U9.7 (~{Y7})
- new net: SW3.2 (B), U9.9 (~{Y6})
- new net PEB: R16.1, SW3.1 (A), U10.23 (CS2B)
- no-connect marks 10 -> 18
Other:
- moved on the sheet: C1, C10, C11, C2, C3, C4, C5, C6, C7, C8, C9, D1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

Commit message: Working on KIM Board
Parts:
- removed J2: VCC, Connector_PinHeader_2.54mm:PinHeader_1x02_P2.54mm_Vertical, symbol Connector_Generic:Conn_01x02
- removed TP1: GND, TestPoint:TestPoint_Pad_2.5x2.5mm, symbol Connector:TestPoint
- removed TP2: VCC, TestPoint:TestPoint_Pad_2.5x2.5mm, symbol Connector:TestPoint
- removed U12: MAX238xNG+, Package_DIP:DIP-24_W7.62mm, symbol Interface_UART:MAX238xNG+
- added C17, C18, C19, C20, C21: 1uF, Capacitor_THT:C_Disc_D5.0mm_W2.5mm_P2.50mm, symbol Device:C
- added J1: RB/WB, Connector_PinHeader_2.54mm:PinHeader_1x02_P2.54mm_Vertical, symbol Connector_Generic:Conn_01x02
- added J10: BUS, Connector_PinHeader_2.54mm:PinHeader_2x20_P2.54mm_Vertical, symbol Connector_Generic:Conn_02x20_Odd_Even
- added J2: IO, Connector_PinHeader_2.54mm:PinHeader_1x08_P2.54mm_Vertical, symbol Connector_Generic:Conn_01x08
- added U11, U13: MAX232, Package_DIP:DIP-16_W7.62mm_Socket_LongPads, symbol Interface_UART:MAX232
- C13: value 1uF -> 100nF
- J3: value POWER LED -> PHI2 EN
- renumbered J9 to J11, J10 to J12, J1 to J4, J4 to J5, J5 to J6, J8 to J7, J6 to J8, J7 to J9, U11 to U12
Connections:
- net $8000: now also J2.1 (Pin_1)
- net $8400: now also J2.2 (Pin_2)
- net $8800: now also J2.3 (Pin_3)
- net $8C00: now also J2.4 (Pin_4)
- net $9000: now also J2.5 (Pin_5)
- net $9400: now also J2.6 (Pin_6)
- net $9800: now also J2.7 (Pin_7)
- net $9C00: now also J2.8 (Pin_8)
- net A0: now also J10.38 (Pin_38)
- net A1: now also J10.36 (Pin_36)
- net A10: now also J10.18 (Pin_18)
- net A11: now also J10.16 (Pin_16)
- net A12: now also J10.14 (Pin_14)
- net A13: now also J10.12 (Pin_12)
- net A14: now also J10.10 (Pin_10)
- net A15: now also J10.8 (Pin_8)
- net A2: now also J10.34 (Pin_34)
- net A3: now also J10.32 (Pin_32)
- net A4: now also J10.30 (Pin_30)
- net A5: now also J10.28 (Pin_28)
- net A6: now also J10.26 (Pin_26)
- net A7: now also J10.24 (Pin_24)
- net A8: now also J10.22 (Pin_22)
- net A9: now also J10.20 (Pin_20)
- net BE: now also J10.11 (Pin_11)
- net CTS: now also U11.8 (R2IN)
- net CTSIN: now also U11.9 (R2OUT)
- net D0: now also J10.37 (Pin_37)
- net D1: now also J10.35 (Pin_35)
- net D2: now also J10.33 (Pin_33)
- net D3: now also J10.31 (Pin_31)
- net D4: now also J10.29 (Pin_29)
- net D5: now also J10.27 (Pin_27)
- net D6: now also J10.25 (Pin_25)
- net D7: now also J10.23 (Pin_23)
- net DCD: now also U13.8 (R2IN)
- net DCDIN: now also U13.9 (R2OUT)
- net DSR: now also U13.13 (R1IN)
- net DSRIN: now also U13.12 (R1OUT)
- net DTR: now also U13.14 (T1OUT)
- net DTROUT: now also U13.11 (T1IN)
- net EXP2: now also J10.21 (Pin_21)
- net EXP3: now also J10.19 (Pin_19)
- net GND: now also C13.2, C17.2, C20.2, C21.2, J10.1 (Pin_1), J10.40 (Pin_40), U11.15 (GND), U13.15 (GND); no longer C15.2
- net HRDB: now also J10.4 (Pin_4), J10.6 (Pin_6)
- net IRQB: now also J10.5 (Pin_5)
- net NMIB: now also J10.7 (Pin_7)
- net PHI2: now also J3.2 (Pin_2), J10.17 (Pin_17); no longer X1.8 (OUT)
- net RB: now also J1.1 (Pin_1)
- net RDY: now also J10.9 (Pin_9)
- net RESB: now also J10.3 (Pin_3)
- net RTS: now also U11.7 (T2OUT)
- net RTSOUT: now also U11.10 (T2IN)
- net RWB: now also J10.13 (Pin_13)
- net RXD: now also U11.13 (R1IN)
- net RXDIN: now also U11.12 (R1OUT)
- net SYNC: now also J10.15 (Pin_15)
- net TXD: now also U11.14 (T1OUT)
- net TXDOUT: now also U11.11 (T1IN)
- net VCC: now also C13.1, J10.2 (Pin_2), J10.39 (Pin_39), U11.16 (VCC), U13.16 (VCC); no longer J3.1 (Pin_1)
- net WB: now also J1.2 (Pin_2)
- net at C15.1: now also U11.4 (C2+)
- net at C16.1: now also U11.2 (VS+)
- net at C14.1: now also U11.1 (C1+)
- net at C14.2: now also U11.3 (C1-)
- net at D1.1 (K), R15.1: no longer J3.2 (Pin_2)
- new net: J3.1 (Pin_1), X1.8 (OUT)
- new net: C15.2, U11.5 (C2-)
- new net: C20.1, U13.2 (VS+)
- new net: C21.1, U13.6 (VS-)
- new net: C18.1, U13.1 (C1+)
- new net: C18.2, U13.3 (C1-)
- new net: C19.1, U13.4 (C2+)
- new net: C19.2, U13.5 (C2-)
- new net: C17.1, U11.6 (VS-)
Other:
- moved on the sheet: C1, C10, C11, C12, C2, C3, C4, C5, C6, C7, C8, C9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
