File: Hardware/KIM Board/Rev 1.0/KIM Board.kicad_pcb (KiCad board)
At the start: 2 copper layers, 280 x 220 mm, 129 parts, among them J1 KIM ENABLE, J2 DB9 FEMALE (DCE), J3 CTS EN, J4 CARD SLOT, J5 6502 BUS, J6 BREADBOARD HEADERS, J7 5V DC, Q1 2N3904, SW1 0, SW10 9, SW11 10, SW12 11, SW13 12, SW14 13, SW15 14, SW16 15, SW17 16, SW18 17, SW19 18, SW2 1, SW20 19, SW21 20, SW22 21, SW23 22, SW24 23, SW25 IO ENABLE, SW26 RESET, SW27 POWER, SW3 2, SW4 3, SW5 4, SW6 5, SW7 6, SW8 7, SW9 8, U1 65C02, U10 74HC138, U11 74HC138, U12 LM555, U13 LCD-16X2, U14 MAX232, U15 R6551AP, U16 MM74C922, U17 74HC00, U2 AS6C62256, U3 AT28C256, U4 74HC00, U5 74HC00, U6 74HC00, U7 74HC138, U8 W65C21N, U9 AT28C64, X1 1 MHz, Y1 1.8432 Mhz

Commit message: KIM Board Rev 1.0 PCB: placement, 3D models, pin-1 dots, schematic links
More of the placement, by hand.

- 3D models: the Cherry MX switches (SW1-SW24) and the ROM's ZIF socket
  (U3) pointed at models KiCad 10 doesn't ship. They now use the ACE's
  CherryMX.step and 228-1277-00-0602J.step, copied into Models, with the
  ACE's offsets: the pads are the same as the ACE's footprints.
- Pin-1 dots: a 0.8 mm dot on the front silkscreen at pin 1 of every IC
  socket, the ZIF and the oscillator, placed as on the ACE: 2.3 mm past
  pin 1 along the row for a DIP, 6.5 mm beside it for the ZIF, 3.8 mm
  past it for the oscillator. U12's sits beside pin 1, clear of its
  label.
- Schematic links: U4, U5, U6, U17 and J6, the multi-unit symbols, had
  no link to the schematic, so Update PCB from Schematic tried to add
  them again. Each now links to its first unit, as KiCad does. The OSHW
  logo is marked board-only, like the other logos.
- The power switch (SW27): its mounting lugs are unnumbered pads, in
  the library and on the board, so Update no longer warns that S1 and
  S2 have no net.

DRC with schematic parity finds no parity issues. Its other reports
are as before: the parts under the LCD, the corner hole in the
breadboards' keep-out, silkscreen warnings on reference labels, and the
unrouted connections.

Co-Authored-By: Claude Opus 5.5 <noreply@anthropic.com>
Parts:
- removed H11, H13, H14, H15, H6: MountingHole, MountingHole:MountingHole_3.2mm_M3
- added G***: LOGO, A.C. Wright Logo:A.C. Wright Logo 10mm, F.Cu at (278.7, 139.4)
- added G***: LOGO, 6502 Logos:6502 KIM Board Logo 5mm, F.Cu at (373.9, 261.2)
- added REF**: OSHW-Logo2_9.8x8mm_SilkScreen, Symbol:OSHW-Logo2_9.8x8mm_SilkScreen, F.Cu at (151.4, 86.0)
- J4: value CARD SLOT -> CART
- J5: value 6502 BUS -> BUS
- moved C17 161.4 mm to (286.8, 168.3), turned to 180 degrees
- moved Q1 124.7 mm to (284.3, 202.2), turned to 180 degrees
- moved R18 123.1 mm to (288.8, 195.0), turned to 180 degrees
- moved R16 118.4 mm to (279.2, 190.1), turned to 90 degrees
- moved D1 116.8 mm to (366.3, 153.5), turned to 180 degrees
- moved C5 110.5 mm to (279.2, 193.7), turned to -90 degrees
- moved C6 109.3 mm to (285.3, 187.6)
- moved U12 109.0 mm to (279.2, 173.0)
- moved R15 101.2 mm to (351.0, 143.9)
- moved SW26 96.9 mm to (267.7, 158.0)
- moved J1 96.5 mm to (361.4, 143.9), turned to 0 degrees
- moved R17 95.1 mm to (273.6, 168.3), turned to 180 degrees
- moved R6 93.6 mm to (185.8, 167.7)
- moved R5 81.0 mm to (135.1, 167.7)
- moved C4 73.8 mm to (360.1, 121.0), turned to 180 degrees
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Other:
- board text added: "$0000"
- board text added: "$8000"
- board text added: "$8400"
- board text added: "$8800"
- board text added: "$8C00"
- board text added: "$9000"
- board text added: "$9400"
- board text added: "$9800"
- board text added: "$9C00"
- board text added: "$C000"
- board text added: "A0"
- board text added: "A1"
- board text added: "A10"
- board text added: "A11"
- board text added: "A12"
- board text added: "A13"
- board text added: "A14"
- board text added: "A15"
- board text added: "A2"
- board text added: "A3"
- board text added: "A4"
- board text added: "A5"
- board text added: "A6"
- board text added: "A7"
- board text added: "A8"
- board text added: "A9"
- board text added: "BE"
- board text added: "D0"
- board text added: "D1"
- board text added: "D2"
- board text added: "D3"
- board text added: "D4"
- board text added: "D5"
- board text added: "D6"
- board text added: "D7"
- board text added: "EXP2"
- board text added: "EXP3"
- board text added: "GND"
- board text added: "GPIO"
- board text added: "HI ROM"
- board text added: "HRDB"
- board text added: "I/O $8000"
- board text added: "IO1"
- board text added: "IO2"
- board text added: "IO3"
- board text added: "IO4"
- board text added: "IO5"
- board text added: "IO6"
- board text added: "IO7"
- board text added: "IO8"
- board text added: "IRQB"
- board text added: "LO ROM $A000"
- board text added: "NMIB"
- board text added: "PHI2"
- board text added: "RAM"
- board text added: "RDY"
- board text added: "RESB"
- board text added: "RTC"
- board text added: "RWB"
- board text added: "SERIAL"
- board text added: "SOUND"
- board text added: "STORAGE"
- board text added: "SYNC"
- board text added: "VCC"
- board text added: "VIDEO"
- board text added: "© 2026 A.C. Wright Design | acwrightdesign.com | Rev 1.0"

Commit message: KIM Board Rev 1.0: pull the PIA's CB1 and CB2 up through R23
CB1 and CB2 are unused, and as CMOS inputs they floated. They are now
joined and held high by one 10k (R23), placed under the LCD. A resistor
rather than a tie to VCC, because software can make CB2 an output.

- Schematic: R23 replaces the two no-connects; the PDF is re-exported.
- PCB: R23 placed, with R15's order fields; the GND pours refilled.
- Tests/check-schematics.mjs checks that CB1 and CB2 are joined and
  have one 10k pull-up.
- README: R23 in the keypad and display bullet, and in the checks.

Co-Authored-By: Claude Opus 5.5 <noreply@anthropic.com>
Parts:
- added R23: 10k, Resistor_THT:R_Axial_DIN0204_L3.6mm_D1.6mm_P5.08mm_Horizontal, F.Cu at (333.0, 121.1)
- moved R17 0.65 mm to (273.6, 167.7)
Connections:
- U8 pad 18: unconnected-(U8-CB1-Pad18) -> Net-(U8-CB1)
- U8 pad 19: unconnected-(U8-CB2-Pad19) -> Net-(U8-CB1)
