File: Hardware/KIM Board/Rev 1.0/KIM Board.kicad_pcb (KiCad board)
At the start: 2 copper layers, 280 x 220 mm, 128 parts, among them J1 KIM ENABLE, J2 DB9 FEMALE (DCE), J3 CTS EN, J4 CART, J5 BUS, J6 BREADBOARD HEADERS, J7 5V DC, Q1 2N3904, SW1 0, SW10 9, SW11 10, SW12 11, SW13 12, SW14 13, SW15 14, SW16 15, SW17 16, SW18 17, SW19 18, SW2 1, SW20 19, SW21 20, SW22 21, SW23 22, SW24 23, SW25 IO ENABLE, SW26 RESET, SW27 POWER, SW3 2, SW4 3, SW5 4, SW6 5, SW7 6, SW8 7, SW9 8, U1 65C02, U10 74HC138, U11 74HC138, U12 LM555, U13 LCD-16X2, U14 MAX232, U15 R6551AP, U16 MM74C922, U17 74HC00, U2 AS6C62256, U3 AT28C256, U4 74HC00, U5 74HC00, U6 74HC00, U7 74HC138, U8 W65C21N, U9 AT28C64, X1 1 MHz, Y1 1.8432 Mhz

Commit message: KIM Board Rev 1.0 PCB: second scripted routing attempt, bus nets only, for reference
The 35 bus nets alone, each pin-to-pin link tried as a fixed shape
(straight with 45-degree jogs, an L with one via, a Z with two).
208 of 235 links routed; the rest were left open. The owner will
route the board by hand instead. Kept here for reference; the next
commit takes it out again.

Co-Authored-By: Claude Opus 5.5 <noreply@anthropic.com>
Routing:
- net RESB: track 0.00 -> 422.3 mm, vias 0 -> 8
- net RWB: track 0.00 -> 381.7 mm, vias 0 -> 7
- net PHI2: track 0.00 -> 380.7 mm, vias 0 -> 12
- net A1: track 0.00 -> 349.1 mm, vias 0 -> 9
- net D3: track 0.00 -> 338.6 mm, vias 0 -> 9
- net D5: track 0.00 -> 328.6 mm, vias 0 -> 9
- net D2: track 0.00 -> 313.8 mm, vias 0 -> 12
- net IRQB: track 0.00 -> 305.1 mm, vias 0 -> 6
- net A11: track 0.00 -> 300.7 mm, vias 0 -> 9
- net D7: track 0.00 -> 291.8 mm, vias 0 -> 15
- net D1: track 0.00 -> 286.6 mm, vias 0 -> 9
- net A2: track 0.00 -> 283.1 mm, vias 0 -> 11
- net A12: track 0.00 -> 277.8 mm, vias 0 -> 7
- net D6: track 0.00 -> 276.8 mm, vias 0 -> 7
- net A9: track 0.00 -> 275.6 mm, vias 0 -> 7
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
Commit message: KIM Board Rev 1.0 PCB: take out the second routing attempt
Back to the unrouted board, for routing by hand. The attempt stays in
the previous commit for reference.

Co-Authored-By: Claude Opus 5.5 <noreply@anthropic.com>
Routing:
- net RESB: track 422.3 -> 0.00 mm, vias 8 -> 0
- net RWB: track 381.7 -> 0.00 mm, vias 7 -> 0
- net PHI2: track 380.7 -> 0.00 mm, vias 12 -> 0
- net A1: track 349.1 -> 0.00 mm, vias 9 -> 0
- net D3: track 338.6 -> 0.00 mm, vias 9 -> 0
- net D5: track 328.6 -> 0.00 mm, vias 9 -> 0
- net D2: track 313.8 -> 0.00 mm, vias 12 -> 0
- net IRQB: track 305.1 -> 0.00 mm, vias 6 -> 0
- net A11: track 300.7 -> 0.00 mm, vias 9 -> 0
- net D7: track 291.8 -> 0.00 mm, vias 15 -> 0
- net D1: track 286.6 -> 0.00 mm, vias 9 -> 0
- net A2: track 283.1 -> 0.00 mm, vias 11 -> 0
- net A12: track 277.8 -> 0.00 mm, vias 7 -> 0
- net D6: track 276.8 -> 0.00 mm, vias 7 -> 0
- net A9: track 275.6 -> 0.00 mm, vias 7 -> 0
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
Commit message: KIM Board Rev 1.0 PCB: first scripted routing attempt, for reference
A first full routing, made by a script that searched a grid of each
part's pin lines: B.Cu horizontal, F.Cu vertical, a via at every turn.
Everything connects and DRC adds no errors, but the owner judged it
far from the ACE's routing: too many vias, above all around the BUS
and CART headers, and lines such as PHI2 forced into detours by lines
routed before them. Kept here for reference; the next commit takes it
out again.

Co-Authored-By: Claude Opus 5.5 <noreply@anthropic.com>
Routing:
- net VCC: track 0.00 -> 1035.4 mm, vias 0 -> 74
- net D5: track 0.00 -> 673.2 mm, vias 0 -> 44
- net A5: track 0.00 -> 602.8 mm, vias 0 -> 36
- net D3: track 0.00 -> 561.5 mm, vias 0 -> 45
- net D6: track 0.00 -> 560.9 mm, vias 0 -> 33
- net D1: track 0.00 -> 474.8 mm, vias 0 -> 34
- net A15: track 0.00 -> 472.0 mm, vias 0 -> 26
- net A13: track 0.00 -> 449.6 mm, vias 0 -> 24
- net A6: track 0.00 -> 441.7 mm, vias 0 -> 36
- net RESB: track 0.00 -> 439.6 mm, vias 0 -> 21
- net A14: track 0.00 -> 439.5 mm, vias 0 -> 31
- net A4: track 0.00 -> 432.2 mm, vias 0 -> 39
- net RWB: track 0.00 -> 425.0 mm, vias 0 -> 23
- net D0: track 0.00 -> 412.1 mm, vias 0 -> 30
- net PHI2: track 0.00 -> 400.4 mm, vias 0 -> 24
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