File: Hardware/KIM Board/Rev 1.0/KIM Board.kicad_pcb (KiCad board)
At the start: 2 copper layers, 280 x 220 mm, 128 parts, among them J1 KIM ENABLE, J2 DB9 FEMALE (DCE), J3 CTS EN, J4 CART, J5 BUS, J6 BREADBOARD HEADERS, J7 5V DC, Q1 2N3904, SW1 0, SW10 9, SW11 10, SW12 11, SW13 12, SW14 13, SW15 14, SW16 15, SW17 16, SW18 17, SW19 18, SW2 1, SW20 19, SW21 20, SW22 21, SW23 22, SW24 23, SW25 IO ENABLE, SW26 RESET, SW27 POWER, SW3 2, SW4 3, SW5 4, SW6 5, SW7 6, SW8 7, SW9 8, U1 65C02, U10 74HC138, U11 74HC138, U12 LM555, U13 LCD-16X2, U14 MAX232, U15 R6551AP, U16 MM74C922, U17 74HC00, U2 AS6C62256, U3 AT28C256, U4 74HC00, U5 74HC00, U6 74HC00, U7 74HC138, U8 W65C21N, U9 AT28C64, X1 1 MHz, Y1 1.8432 Mhz

Commit message: KIM Board Rev 1.0 PCB: routing in progress
The owner's hand routing so far: 1022 track segments and 195 vias.

Co-Authored-By: Claude Opus 5.5 <noreply@anthropic.com>
Parts:
- moved C13 0.38 mm to (307.2, 153.4)
Routing:
- net VCC: track 0.00 -> 1190.4 mm, vias 0 -> 51
- net IRQB: track 0.00 -> 284.8 mm, vias 0 -> 6
- net PHI2: track 0.00 -> 136.4 mm, vias 0 -> 2
- net RWB: track 0.00 -> 134.4 mm, vias 0 -> 3
- net BE: track 0.00 -> 107.4 mm, vias 0 -> 2
- net Net-(U13-VO): track 0.00 -> 102.4 mm, vias 0 -> 3
- net RDY: track 0.00 -> 99.7 mm, vias 0 -> 2
- net D4: track 0.00 -> 99.3 mm, vias 0 -> 3
- net D6: track 0.00 -> 99.2 mm, vias 0 -> 3
- net D5: track 0.00 -> 99.2 mm, vias 0 -> 3
- net PA4: track 0.00 -> 96.9 mm, vias 0 -> 4
- net NMIB: track 0.00 -> 88.7 mm, vias 0 -> 2
- net CA2: track 0.00 -> 76.7 mm, vias 0 -> 4
- net SYNC: track 0.00 -> 74.3 mm, vias 0 -> 1
- net A0: track 0.00 -> 71.8 mm, vias 0 -> 4
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
Commit message: KIM Board Rev 1.0: label the keypad switches with their KIM keys
The 24 matrix switches carried their keycodes (0-23) as values, which
only matched the key for 1-9. Each now carries the key the KC Monitor
gives that keycode (kim.inc): SW1 LEFT, SW11 0, SW12 RIGHT, SW13-SW16
F E D C, SW17 ESC, SW18 INS, SW19 PGUP, SW20 A, SW21 UP, SW22 DEL,
SW23 PGDN, SW24 B.

- Schematic and PCB: the values changed, nothing else; schematic
  parity is clean.
- The schematic PDF is re-exported.

Co-Authored-By: Claude Opus 5.5 <noreply@anthropic.com>
Parts:
- SW1: value 0 -> LEFT
- SW11: value 10 -> 0
- SW12: value 11 -> RIGHT
- SW13: value 12 -> F
- SW14: value 13 -> E
- SW15: value 14 -> D
- SW16: value 15 -> C
- SW17: value 16 -> ESC
- SW18: value 17 -> INS
- SW19: value 18 -> PGUP
- SW20: value 19 -> A
- SW21: value 20 -> UP
- SW22: value 21 -> DEL
- SW23: value 22 -> PGDN
- SW24: value 23 -> B
Changed lines of the file:
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@@
 			)
 		)
-		(property "Value" "15"
+		(property "Value" "C"
 			(at -2.54 12.954 0)
 			(layer "F.SilkS")
@@
 			)
 		)
-		(property "Value" "13"
+		(property "Value" "E"
 			(at -2.54 12.954 0)
 			(layer "F.SilkS")
@@
 			)
 		)
-		(property "Value" "10"
+		(property "Value" "0"
 			(at -2.54 12.954 0)
 			(layer "F.SilkS")
@@
 			)
 		)
-		(property "Value" "16"
+		(property "Value" "ESC"
 			(at -2.54 12.954 0)
 			(layer "F.SilkS")
@@
 			)
 		)
-		(property "Value" "14"
+		(property "Value" "D"
 			(at -2.54 12.954 0)
 			(layer "F.SilkS")
@@
 			)
 		)
-		(property "Value" "20"
+		(property "Value" "UP"
 			(at -2.54 12.954 0)
 			(layer "F.SilkS")
@@
 			)
 		)
-		(property "Value" "22"
+		(property "Value" "PGDN"
 			(at -2.54 12.954 0)
 			(layer "F.SilkS")
@@
 			)
 		)
-		(property "Value" "18"
+		(property "Value" "PGUP"
 			(at -2.54 12.954 0)
 			(layer "F.SilkS")
@@
 			)
 		)
-		(property "Value" "21"
+		(property "Value" "DEL"
 			(at -2.54 12.954 0)
 			(layer "F.SilkS")
@@
 			)
 		)
-		(property "Value" "17"
+		(property "Value" "INS"
 			(at -2.54 12.954 0)
 			(layer "F.SilkS")
@@
 			)
 		)
-		(property "Value" "12"
+		(property "Value" "F"
 			(at -2.54 12.954 0)
 			(layer "F.SilkS")
@@
 			)
 		)
-		(property "Value" "11"
+		(property "Value" "RIGHT"
 			(at -2.54 12.954 0)
 			(layer "F.SilkS")
@@
 			)
 		)
-		(property "Value" "19"
+		(property "Value" "A"
 			(at -2.54 12.954 0)
 			(layer "F.SilkS")
@@
 			)
 		)
-		(property "Value" "0"
+		(property "Value" "LEFT"
 			(at -2.54 12.954 0)
 			(layer "F.SilkS")
@@
 			)
 		)
-		(property "Value" "23"
+		(property "Value" "B"
 			(at -2.54 12.954 0)
 			(layer "F.SilkS")

Commit message: KIM Board Rev 1.0: arrows for the keypad's LEFT, RIGHT and UP keys
SW1, SW12 and SW21 now carry ←, → and ↑ in place of LEFT, RIGHT and
UP, on the schematic and the PCB's silkscreen. KiCad's stroke font
draws all three. Schematic parity is clean, and the schematic PDF is
re-exported.

Co-Authored-By: Claude Opus 5.5 <noreply@anthropic.com>
Parts:
- SW1: value LEFT -> ←
- SW12: value RIGHT -> →
- SW21: value UP -> ↑
Changed lines of the file:
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@@
 			)
 		)
-		(property "Value" "UP"
+		(property "Value" "↑"
 			(at -2.54 12.954 0)
 			(layer "F.SilkS")
@@
 			)
 		)
-		(property "Value" "RIGHT"
+		(property "Value" "→"
 			(at -2.54 12.954 0)
 			(layer "F.SilkS")
@@
 			)
 		)
-		(property "Value" "LEFT"
+		(property "Value" "←"
 			(at -2.54 12.954 0)
 			(layer "F.SilkS")
