File: Hardware/Keypad Card/Rev 1.0/Keypad Card.kicad_pcb (KiCad board)
At the start: 2 copper layers, 100 x 57.6 mm, 14 parts, among them J1 6502 Card Edge, J2 PORT A, J3 PORT B, U1 74HC138, U2 74HC138, U3 65C21, U4 AT28C64

Commit message: Finish Keypad Card
Parts:
- moved C4 0.44 mm to (128.3, 98.9)
Connections:
- J1 pad EXP0: unconnected-(J1-PadEXP0) -> GND
- J1 pad EXP1: unconnected-(J1-PadEXP1) -> GND
Routing:
- net VCC: track 0.00 -> 210.6 mm, vias 0 -> 8
- net CB2: track 0.00 -> 99.1 mm, vias 0 -> 3
- net CB1: track 0.00 -> 91.8 mm, vias 0 -> 3
- net IRQB: track 0.00 -> 86.1 mm, vias 0 -> 2
- net RESB: track 0.00 -> 82.6 mm, vias 0 -> 4
- net PB3: track 0.00 -> 80.7 mm, vias 0 -> 3
- net PHI2: track 0.00 -> 79.2 mm, vias 0 -> 7
- net PB6: track 0.00 -> 79.1 mm, vias 0 -> 3
- net PB5: track 0.00 -> 79.1 mm, vias 0 -> 3
- net PB7: track 0.00 -> 79.0 mm, vias 0 -> 3
- net PB4: track 0.00 -> 79.0 mm, vias 0 -> 3
- net PB2: track 0.00 -> 75.7 mm, vias 0 -> 3
- net RWB: track 0.00 -> 72.7 mm, vias 0 -> 4
- net PB1: track 0.00 -> 70.5 mm, vias 0 -> 3
- net PB0: track 0.00 -> 65.5 mm, vias 0 -> 3
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